File: pcb/yuletronics.kicad_pcb (KiCad board)
At the start: 2 copper layers, 45 x 50 mm, 35 parts, among them IC1 STM32F042F6P6, IC2 MCP1700, IC3 TLV61225, J1 BATT, J2 MICROUSB, P1 SWD_TC, SW1 BOOTLOAD, SW2 PWR_SWITCH

Commit message: Added ESP
Parts:
- added R12: 10k, agg:0805, F.Cu at (125.4, 113.5)
- added R13: 10k, agg:0805, F.Cu at (125.4, 108.9)
- added R14: 10k, agg:0805, F.Cu at (125.4, 111.2)
- added U1: ESP8266-ESP01, agg:ESP8266-ESP01, F.Cu at (97.5, 118.0)
- SW1: value BOOTLOAD -> PRG
- moved R1 17.0 mm to (125.4, 106.6)
- moved R4 7.78 mm to (115.1, 119.9)
- turned D1 to 243.4 degrees
Connections:
- IC1 pad 1: /SWITCH -> Net-(IC1-Pad1)
- IC1 pad 2: Net-(IC1-Pad2) -> /LED2
- IC1 pad 3: Net-(IC1-Pad3) -> /LED3
- IC1 pad 7: /LED2 -> /LED4
- IC1 pad 8: /LED3 -> /USART2_TX
- IC1 pad 9: /LED4 -> /USART2_RX
- R1 pad 1: /SWITCH -> 3v3
- R1 pad 2: GND -> Net-(R1-Pad2)
- SW1 pad 1: 3v3 -> GND
- SW1 pad 2: /SWITCH -> Net-(R1-Pad2)
Routing:
- net /USART2_TX: track 0.00 -> 24.1 mm, vias 0 -> 1
- net Net-(R1-Pad2): track 0.00 -> 22.3 mm
- net 3v3: track 63.9 -> 81.4 mm, vias 2 -> 4
- net /SWITCH: track 15.8 -> 0.00 mm
- net GND: track 31.6 -> 46.0 mm, vias 18 -> 19
- net /USART2_RX: track 0.00 -> 11.8 mm, vias 0 -> 1
- net Net-(U1-Pad16): track 8.93 -> 0.00 mm
- net 5v: track 14.0 -> 23.0 mm
- net Net-(D1-Pad2): track 2.32 -> 8.15 mm
- net Net-(R14-Pad1): track 0.00 -> 4.46 mm
- net Net-(R13-Pad1): track 0.00 -> 4.36 mm
- net /LED3: track 28.7 -> 25.3 mm
- net /LED2: track 25.4 -> 22.1 mm
- net Net-(IC1-Pad1): track 0.00 -> 2.53 mm
- net /LED1: track 14.4 -> 11.9 mm
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