File: pcb/yuletronics.kicad_pcb (KiCad board)
At the start: 2 copper layers, 45 x 50 mm, 39 parts, among them IC1 STM32F042F6P6, IC2 MCP1700, IC3 TLV61225, J1 BATT, J2 MICROUSB, P1 SWD_TC, SW1 PRG, SW2 PWR_SWITCH, U1 ESP8266-ESP01

Commit message: Final Changes
Parts:
- U1: moved to B.Cu
- moved U1 43.6 mm to (141.1, 118.2), turned to 180 degrees
- moved R14 4.80 mm to (125.4, 106.4), turned to 180 degrees
- moved R1 4.60 mm to (125.4, 111.2)
- moved R13 0.10 mm to (125.4, 108.8)
Routing:
- net GND: track 46.0 -> 32.8 mm, vias 19 -> 18
- net Net-(R14-Pad1): track 4.46 -> 17.3 mm
- net /USART2_TX: track 24.1 -> 19.7 mm
- net Net-(R1-Pad2): track 22.3 -> 18.3 mm
- net Net-(R13-Pad1): track 4.36 -> 6.92 mm
- net /USART2_RX: track 11.8 -> 13.1 mm
- net 3v3: track 81.4 -> 82.7 mm
Other:
- board text added: "MCoates"
- board text added: "evil"
- board text added: "tree"
